Commit message: Update: tempertature

File: urdf/fishbot_base.urdf (robot description, URDF)
Before this commit: robot fishbot, 9 links, 8 joints
Links:
- added link temperature_test_link, mass 0.1; collision box size=0.02 0.02 0.02; visual box size=0.02 0.02 0.02
Joints:
- added joint temperature_test_joint: type fixed, parent base_link, child temperature_test_link, origin xyz=0 0 0.02
